File: hardware/BuckPower.kicad_sch (KiCad schematic)
At the start: 31 parts, among them Q401 2N7002NXAKR, U401 SIC437A

Commit message: Exchanged 5k11 with 5k1 part number
Parts:
- R401, R405: ManufacturerNumber RT0603DRE075K11L -> RC0603FR-105K1L; MouserNumber 603-RT0603DRE075K11L -> 603-RC0603FR-105K1L
Changed lines of the file:
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@@
 			)
 		)
-		(property "MouserNumber" "603-RT0603DRE075K11L"
+		(property "MouserNumber" "603-RC0603FR-105K1L"
 			(at 69.85 58.42 0)
 			(effects
@@
 			)
 		)
-		(property "ManufacturerNumber" "RT0603DRE075K11L"
+		(property "ManufacturerNumber" "RC0603FR-105K1L"
 			(at 69.85 58.42 90)
 			(effects
@@
 			)
 		)
-		(property "MouserNumber" "603-RT0603DRE075K11L"
+		(property "MouserNumber" "603-RC0603FR-105K1L"
 			(at 53.34 34.29 0)
 			(effects
@@
 			)
 		)
-		(property "ManufacturerNumber" "RT0603DRE075K11L"
+		(property "ManufacturerNumber" "RC0603FR-105K1L"
 			(at 53.34 34.29 90)
 			(effects
